Commit message: Updated files

File: urdf/m2wr.xacro (robot description, xacro)
@@ -4,5 +4,5 @@
   <xacro:include filename="$(find vacbot)/urdf/m2wr.gazebo" />
   <xacro:include filename="$(find vacbot)/urdf/macros.xacro" />
-  <link name="link_chassis">
+  <link name="base_link">
     <!-- pose and inertial -->
     <pose>0 0 0.1 0 0 0</pose>
@@ -71,5 +71,5 @@
   <joint name="joint_sensor_laser" type="fixed">
     <origin xyz="0.15 0 0.05" rpy="0 0 0"/>
-    <parent link="link_chassis"/>
+    <parent link="base_link"/>
     <child link="sensor_laser"/>
   </joint>

File: urdf/macros.xacro (robot description, xacro)
@@ -26,5 +26,5 @@
         <origin rpy="0 0 0" xyz="${origin_xyz}"/>
         <child link="${child}"/>
-        <parent link="link_chassis"/>
+        <parent link="base_link"/>
         <axis rpy="0 0 0" xyz="0 1 0"/>
         <limit effort="10000" velocity="1000"/>
